Commit message: more changes to templates

File: templates/package_properties.xacro (robot description, xacro)
@@ -7,6 +7,5 @@
 	   <xacro:arg name="static" default="true"/>
        <!-- Package of this model -->
-	   <xacro:property name="package"  default="###PACKAGE###" />
-	   <xacro:property name="meshdir"  default="###MESH_DIR###" />
+	   <xacro:property name="ros_package"  default="###PACKAGE###" />
 	   <xacro:if value="$(arg static)">
 			<gazebo>

File: templates/template_simple.xacro (robot description, xacro)
@@ -4,51 +4,55 @@
        xmlns:interface="http://playerstage.sourceforge.net/gazebo/xmlschema/#interface"
        xmlns:xacro="http://ros.org/wiki/xacro" name="###MODEL_NAME###">
-      <xacro:include filename="basic/package_properties.xacro"/>
-      <!-- #################################################################################### -->
-      <!-- #These are the default values for each object, it is recommended to change the here# -->
-      <!-- #################################################################################### -->
-	  <!-- if the mesh collision is prefered to the simplyfied autogenerated one -->
-	  <xacro:arg name="mesh_collision" default="false" />
-	  <!-- the scaling of the object -->
-	  <xacro:arg name="scale_x" default="###SCALE_X###" />
-	  <xacro:arg name="scale_y" default="###SCALE_Y###" />
-	  <xacro:arg name="scale_z" default="###SCALE_Z###" />
-	  <!-- Inertial of the model -->
-	  <xacro:arg name="mass" 	 default="###MASS###" />
-	  <xacro:arg name="ixx" default="###INERTIA_XX###" />
-	  <xacro:arg name="ixy" default="###INERTIA_XY###" />
-	  <xacro:arg name="ixz" default="###INERTIA_XZ###" />
-	  <xacro:arg name="iyy" default="###INERTIA_YY###" />
-	  <xacro:arg name="iyz" default="###INERTIA_YZ###" />
-	  <xacro:arg name="izz" default="###INERTIA_ZZ###" />
-	  <xacro:property name="meshfile" default="###MESH_FILE###" />
-<!--
-<link name="###OBJ_NAME###">
-        <visual>
-                <geometry>
-        			<mesh filename="package://${package}/${mesh_dir}/${mesh_file}"/>
-                </geometry>
-        </visual>
-        <collision>
-        	<xacro:if value="$(arg mesh_collision)" >
-        		<geometry>
-					<mesh filename="package://${package}/${mesh_dir}/${mesh_file}"/>
-                </geometry>
-        	</xacro:if>
-        	<xacro:if value="${$(arg mesh_collision) == false}" >
-        		<geometry>
-					###SIMPLE_COLLISIONS###
-                </geometry>
-        	</xacro:if>
-        </collision>
-	<inertial>
-		<mass value="$(arg mass)" />
-		<inertia ixx="$(arg ixx)"
-				 ixy="$(arg ixy)"
-				 ixz="$(arg ixz)"
-				 iyy="$(arg iyy)"
-				 izz="$(arg izz)" />
-	</inertial>
-</link>
-       	-->
+		<xacro:include filename="basic/package_properties.xacro"/>
+		<!-- #################################################################################### -->
+		<!-- #These are the default values for each object, it is recommended to change the here# -->
+		<!-- #################################################################################### -->
+		<!-- if the mesh collision is prefered to the simplyfied autogenerated one -->
+		<xacro:arg name="mesh_collision" default="false" />
+		<!-- the scaling of the object -->
+		<xacro:arg name="scale_x" default="###SCALE_X###" />
+		<xacro:arg name="scale_y" default="###SCALE_Y###" />
+		<xacro:arg name="scale_z" default="###SCALE_Z###" />
+		<!-- Inertial of the model -->
+		<xacro:arg name="mass" 	 default="###MASS###" />
+		<xacro:arg name="ixx" default="###INERTIA_XX###" />
+		<xacro:arg name="ixy" default="###INERTIA_XY###" />
+		<xacro:arg name="ixz" default="###INERTIA_XZ###" />
+		<xacro:arg name="iyy" default="###INERTIA_YY###" />
+		<xacro:arg name="iyz" default="###INERTIA_YZ###" />
+		<xacro:arg name="izz" default="###INERTIA_ZZ###" />
+		<xacro:property name="elevation" default="###ELEVATION###" />
+		<xacro:property name="meshfile" value="###MESH_FILE###" />
+		<xacro:property name="model_name" value="###MODEL_NAME###" />
+		<link name="${model_name}_base_link"/>
+		<joint name="joint_fixed_${model_name}_base_link_${model_name}" type="fixed">
+			<origin xyz="${elevation}" />
+			<parent link="${model_name}_base_link" />
+			<child  link="${model_name}" />
+		</joint>
+		<link name="${model_name}">
+		    <visual>
+		            <geometry>
+		    			<mesh filename="${meshfile}"/>
+		            </geometry>
+		    </visual>
+		    <collision>
+		    	<xacro:if value="$(arg mesh_collision)" >
+		    		<geometry>
+						<mesh filename="${meshfile}"/>
+		            </geometry>
+		    	</xacro:if>
+		    	<xacro:if value="${$(arg mesh_collision) == false}" >
+						###SIMPLE_COLLISIONS###
+		    	</xacro:if>
+		    </collision>
+		<inertial>
+			<mass value="$(arg mass)" />
+			<inertia ixx="$(arg ixx)"
+					 ixy="$(arg ixy)"
+					 ixz="$(arg ixz)"
+					 iyy="$(arg iyy)"
+					 izz="$(arg izz)" />
+		</inertial>
+		</link>
 </robot>

Commit message: remove stuff from main template
will probably be removed

File: templates/package_properties.xacro (robot description, xacro)
@@ -4,12 +4,3 @@
        xmlns:interface="http://playerstage.sourceforge.net/gazebo/xmlschema/#interface"
        xmlns:xacro="http://ros.org/wiki/xacro" >
-       <!-- if object is static not movable by actors -->
-	   <xacro:arg name="static" default="true"/>
-       <!-- Package of this model -->
-	   <xacro:property name="ros_package"  default="###PACKAGE###" />
-	   <xacro:if value="$(arg static)">
-			<gazebo>
-			    <static>true</static>
-			</gazebo>
-	   </xacro:if>
 </root>
