Commit message: add changes to template

File: templates/template_simple.xacro (robot description, xacro)
@@ -8,4 +8,11 @@
 		<!-- #These are the default values for each object, it is recommended to change the here# -->
 		<!-- #################################################################################### -->
+	   <!-- if object is static not movable by actors -->
+	   <xacro:arg name="static" default="true"/>
+	   <xacro:if value="$(arg static)">
+			<gazebo>
+			    <static>true</static>
+			</gazebo>
+	   </xacro:if>
 		<!-- if the mesh collision is prefered to the simplyfied autogenerated one -->
 		<xacro:arg name="mesh_collision" default="false" />
@@ -22,10 +29,11 @@
 		<xacro:arg name="iyz" default="###INERTIA_YZ###" />
 		<xacro:arg name="izz" default="###INERTIA_ZZ###" />
-		<xacro:property name="elevation" default="###ELEVATION###" />
-		<xacro:property name="meshfile" value="###MESH_FILE###" />
-		<xacro:property name="model_name" value="###MODEL_NAME###" />
+        <!-- Package of this model -->
+		<xacro:property name="elevate" 		value="###ELEVATION###" />
+		<xacro:property name="meshfile" 	value="###MESH_FILE###" />
+		<xacro:property name="model_name" 	value="###MODEL_NAME###" />
 		<link name="${model_name}_base_link"/>
 		<joint name="joint_fixed_${model_name}_base_link_${model_name}" type="fixed">
-			<origin xyz="${elevation}" />
+			<origin xyz="0 0 ${-elevate}" />
 			<parent link="${model_name}_base_link" />
 			<child  link="${model_name}" />

Commit message: fix inertia in template

File: templates/template_simple.xacro (robot description, xacro)
@@ -16,5 +16,5 @@
 	   </xacro:if>
 		<!-- if the mesh collision is prefered to the simplyfied autogenerated one -->
-		<xacro:arg name="mesh_collision" default="false" />
+		<xacro:arg name="mesh_collision" default="False" />
 		<!-- the scaling of the object -->
 		<xacro:arg name="scale_x" default="###SCALE_X###" />
@@ -23,10 +23,10 @@
 		<!-- Inertial of the model -->
 		<xacro:arg name="mass" 	 default="###MASS###" />
-		<xacro:arg name="ixx" default="###INERTIA_XX###" />
-		<xacro:arg name="ixy" default="###INERTIA_XY###" />
-		<xacro:arg name="ixz" default="###INERTIA_XZ###" />
-		<xacro:arg name="iyy" default="###INERTIA_YY###" />
-		<xacro:arg name="iyz" default="###INERTIA_YZ###" />
-		<xacro:arg name="izz" default="###INERTIA_ZZ###" />
+		<xacro:arg name="ixx"    default="###INERTIA_XX###" />
+		<xacro:arg name="ixy"    default="###INERTIA_XY###" />
+		<xacro:arg name="ixz"    default="###INERTIA_XZ###" />
+		<xacro:arg name="iyy"    default="###INERTIA_YY###" />
+		<xacro:arg name="iyz"    default="###INERTIA_YZ###" />
+		<xacro:arg name="izz"    default="###INERTIA_ZZ###" />
         <!-- Package of this model -->
 		<xacro:property name="elevate" 		value="###ELEVATION###" />
@@ -42,5 +42,5 @@
 		    <visual>
 		            <geometry>
-		    			<mesh filename="${meshfile}"/>
+		    			<mesh filename="${meshfile}" scale="$(arg scale_x) $(arg scale_y) $(arg scale_z)"/>
 		            </geometry>
 		    </visual>
@@ -51,7 +51,7 @@
 		            </geometry>
 		    	</xacro:if>
-		    	<xacro:if value="${$(arg mesh_collision) == false}" >
+		    	<xacro:unless value="$(arg mesh_collision)" >
 						###SIMPLE_COLLISIONS###
-		    	</xacro:if>
+		    	</xacro:unless>
 		    </collision>
 		<inertial>
@@ -61,5 +61,7 @@
 					 ixz="$(arg ixz)"
 					 iyy="$(arg iyy)"
-					 izz="$(arg izz)" />
+				     iyz="$(arg iyz)"
+					 izz="$(arg izz)"
+					/>
 		</inertial>
 		</link>

Commit message: fix elevation and scaling

File: templates/template_simple.xacro (robot description, xacro)
@@ -35,5 +35,5 @@
 		<link name="${model_name}_base_link"/>
 		<joint name="joint_fixed_${model_name}_base_link_${model_name}" type="fixed">
-			<origin xyz="0 0 ${-elevate}" />
+			<origin xyz="0 0 ${-elevate*$(arg scale_z)}" />
 			<parent link="${model_name}_base_link" />
 			<child  link="${model_name}" />
